File: kicad/pal2rom.kicad_pcb (KiCad board)
At the start: 2 copper layers, 85 x 100 mm, 11 parts, among them J1 PAL2_Expansion, J4 RIOT+, U1 28C256, U2 74LS145

Commit message: Minor improvements
Routing:
- net /A000-BFFF: track 21.4 -> 31.4 mm
- net /C000-DFFF: track 21.4 -> 27.3 mm
- net /E000-FFFF: track 29.6 -> 30.5 mm
Other:
- board text added: "PAL-2 ROM Whatsit Plastic Objects Limited"
- board text removed: "Plastic Objects Limited"
Changed lines of the file:
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@@
 		)
 	)
-	(gr_text "Plastic Objects Limited"
-		(at 160.02 138.6915 0)
+	(gr_text "PAL-2 ROM Whatsit\nPlastic Objects Limited"
+		(at 152.908 138.6915 0)
 		(layer "B.SilkS")
 		(effects
 			(font
-				(size 2.5 2.5)
-				(thickness 0.3)
-				(bold yes)
+				(size 2 2)
+				(thickness 0.1875)
 			)
 			(justify left bottom mirror)
@@
 	)
 	(gr_text "Rev 0 - 10/2026"
-		(at 83.566 138.684 0)
+		(at 88.138 138.684 0)
 		(layer "B.SilkS")
 		(effects
@@
 	)
 	(segment
-		(start 124.968 103.632)
+		(start 107.95 108.331)
+		(end 109.347 109.728)
+		(width 0.2)
+		(layer "B.Cu")
+		(net 46)
+	)
+	(segment
+		(start 123.444 109.728)
+		(end 124.46 108.712)
+		(width 0.2)
+		(layer "B.Cu")
+		(net 46)
+	)
+	(segment
+		(start 124.46 108.712)
+		(end 124.46 104.14)
+		(width 0.2)
+		(layer "B.Cu")
+		(net 46)
+	)
+	(segment
+		(start 107.95 104.394)
+		(end 107.95 108.331)
+		(width 0.2)
+		(layer "B.Cu")
+		(net 46)
+	)
+	(segment
+		(start 105.918 102.362)
+		(end 107.95 104.394)
+		(width 0.2)
+		(layer "B.Cu")
+		(net 46)
+	)
+	(segment
+		(start 124.46 104.14)
 		(end 126.238 102.362)
 		(width 0.2)
@@
 	)
 	(segment
-		(start 105.918 102.362)
-		(end 107.188 103.632)
+		(start 109.347 109.728)
+		(end 123.444 109.728)
 		(width 0.2)
 		(layer "B.Cu")
@@
 	)
 	(segment
-		(start 107.188 103.632)
-		(end 123.952 103.632)
-		(width 0.2)
-		(layer "B.Cu")
-		(net 46)
-	)
-	(segment
-		(start 123.952 103.632)
-		(end 124.968 103.632)
-		(width 0.2)
-		(layer "B.Cu")
-		(net 46)
+		(start 130.772 110.528)
+		(end 133.858 107.442)
+		(width 0.2)
+		(layer "B.Cu")
+		(net 47)
 	)
 	(segment
 		(start 105.918 107.442)
-		(end 107.95 109.474)
-		(width 0.2)
-		(layer "F.Cu")
+		(end 109.004 110.528)
+		(width 0.2)
+		(layer "B.Cu")
 		(net 47)
 	)
 	(segment
-		(start 107.95 109.474)
-		(end 131.826 109.474)
-		(width 0.2)
-		(layer "F.Cu")
+		(start 109.004 110.528)
+		(end 130.772 110.528)
+		(width 0.2)
+		(layer "B.Cu")
 		(net 47)
 	)
 	(segment
-		(start 131.826 109.474)
-		(end 133.858 107.442)
-		(width 0.2)
-		(layer "F.Cu")
-		(net 47)
-	)
-	(segment
-		(start 124.968 106.172)
-		(end 122.428 106.172)
+		(start 109.181315 110.128)
+		(end 123.609686 110.128)
 		(width 0.2)
 		(layer "B.Cu")
@@
 	)
 	(segment
-		(start 122.428 106.172)
-		(end 107.188 106.172)
+		(start 124.86 106.28)
+		(end 126.238 104.902)
 		(width 0.2)
 		(layer "B.Cu")
@@
 	)
 	(segment
-		(start 126.238 104.902)
-		(end 124.968 106.172)
+		(start 123.609686 110.128)
+		(end 124.86 108.877685)
 		(width 0.2)
 		(layer "B.Cu")
@@
 	(segment
 		(start 105.918 104.902)
-		(end 107.188 106.172)
+		(end 107.55 106.534)
+		(width 0.2)
+		(layer "B.Cu")
+		(net 48)
+	)
+	(segment
+		(start 107.55 106.534)
+		(end 107.55 108.496686)
+		(width 0.2)
+		(layer "B.Cu")
+		(net 48)
+	)
+	(segment
+		(start 124.86 108.877685)
+		(end 124.86 106.28)
+		(width 0.2)
+		(layer "B.Cu")
+		(net 48)
+	)
+	(segment
+		(start 107.55 108.496686)
+		(end 109.181315 110.128)
 		(width 0.2)
 		(layer "B.Cu")
@@
 		(end 154.432 109.474)
 		(width 0.2)
-		(layer "B.Cu")
+		(layer "F.Cu")
 		(net 56)
 	)
@@
 		(end 155.448 117.602)
 		(width 0.2)
-		(layer "B.Cu")
+		(layer "F.Cu")
 		(net 56)
 	)
@@
 		(end 155.448 110.49)
 		(width 0.2)
-		(layer "B.Cu")
+		(layer "F.Cu")
 		(net 56)
 	)
@@
 		(end 120.65 109.474)
 		(width 0.2)
-		(layer "B.Cu")
+		(layer "F.Cu")
 		(net 56)
 	)

Commit message: Fix CS/OS issues
Parts:
- added C3: .1uF, Capacitor_THT:C_Disc_D5.0mm_W2.5mm_P2.50mm, F.Cu at (139.4, 85.3)
- added R1: 1K2, Resistor_THT:R_Axial_DIN0207_L6.3mm_D2.5mm_P7.62mm_Horizontal, F.Cu at (111.0, 49.0)
- added U3: 74LS04, Package_DIP:DIP-14_W7.62mm, F.Cu at (131.8, 89.7)
- U2: footprint Package_DIP:DIP-16_W7.62mm_Socket -> Package_DIP:DIP-16_W7.62mm
- moved C1 12.9 mm to (126.2, 85.3), turned to 180 degrees
- moved JP1 7.62 mm to (95.8, 102.4)
- moved JP2 7.62 mm to (108.5, 84.6)
- moved JP3 7.62 mm to (98.3, 84.6)
- moved U2 7.62 mm to (118.6, 89.7)
- moved JP4 7.62 mm to (111.0, 102.4)
Connections:
- JP1 pad 1: /~{OE} -> /~{CS}
- JP1 pad 3: /~{OE} -> /~{CS}
- JP1 pad 5: /~{OE} -> /~{CS}
- JP2 pad 4: /AB13 -> Net-(JP2-Pin_4)
- JP4 pad 1: /~{OE} -> /~{CS}
- JP4 pad 2: /~{CS} -> /~{OE}
Routing:
- net /AB14: track 34.8 -> 66.5 mm
- net /AB15: track 31.8 -> 62.3 mm
- net VCC: track 109.6 -> 139.1 mm
- net /~{OE}: track 112.1 -> 86.6 mm
- net Net-(JP2-Pin_4): track 0.00 -> 22.9 mm
- net /AB13: track 57.1 -> 39.7 mm
- net /~{CS}: track 101.1 -> 115.4 mm
- net /A13: track 126.2 -> 133.0 mm
- net /8K7_ROM: track 45.2 -> 51.2 mm
- net /A14: track 20.2 -> 16.3 mm
- net /AB9: track 96.5 -> 95.9 mm
Other:
- board text added: "ROM BANK"
- board text added: "Rev 1 - 10/2026"
- board text removed: "ROM CONFIG"
- board text removed: "Rev 0 - 10/2026"
