File: kicad/pal2rom.kicad_sch (KiCad schematic)
At the start: 10 parts, among them J1 PAL2_Expansion, J4 RIOT+, U1 28C256, U2 74LS145

Commit message: Fix CS/OS issues
Parts:
- added C3: .1uF, Capacitor_THT:C_Disc_D5.0mm_W2.5mm_P2.50mm, symbol Device:C_Small
- added R1: 1K2, Resistor_THT:R_Axial_DIN0207_L6.3mm_D2.5mm_P7.62mm_Horizontal, symbol Device:R_US
- added U3: 74LS04, Package_DIP:DIP-14_W7.62mm, symbol 74xx:74LS04
- U2: footprint Package_DIP:DIP-16_W7.62mm_Socket -> Package_DIP:DIP-16_W7.62mm
Connections:
- net AB13: now also U3.1; no longer JP2.4 (Pin_4)
- net GND: now also C3.2, U3.11, U3.13, U3.3, U3.5, U3.7 (GND), U3.9
- net VCC: now also C3.1, R1.1, U3.14 (VCC)
- net ~{CS}: now also JP1.1 (Pin_1), JP1.3 (Pin_3), JP1.5 (Pin_5), JP4.1 (Pin_1), R1.2; no longer JP4.2 (Pin_2)
- net ~{OE}: now also JP4.2 (Pin_2); no longer JP1.1 (Pin_1), JP1.3 (Pin_3), JP1.5 (Pin_5), JP4.1 (Pin_1)
- new net: JP2.4 (Pin_4), U3.2
- no-connect marks 40 -> 45
Other:
- moved on the sheet: C1, C2, JP2, JP3, JP4
