File: kicad/pal2rom.kicad_sch (KiCad schematic)
At the start: 10 parts, among them J1 PAL2_Expansion, J4 RIOT+, U1 28C256, U2 74LS145

Commit message: Improve addressing
Parts:
- added C2: .1uF, Capacitor_THT:C_Disc_D5.0mm_W2.5mm_P2.50mm, symbol Device:C_Small
- added JP5: A13_INV, Connector_PinHeader_2.54mm:PinHeader_1x03_P2.54mm_Vertical, symbol Connector_Generic:Conn_01x03
- added JP6: A12_INV, Connector_PinHeader_2.54mm:PinHeader_1x03_P2.54mm_Vertical, symbol Connector_Generic:Conn_01x03
- added JP7: A11_INV, Connector_PinHeader_2.54mm:PinHeader_1x03_P2.54mm_Vertical, symbol Connector_Generic:Conn_01x03
- added R1: 1K2, Resistor_THT:R_Axial_DIN0207_L6.3mm_D2.5mm_P7.62mm_Horizontal, symbol Device:R_US
- added U3: 74LS04, Package_DIP:DIP-14_W7.62mm, symbol 74xx:74LS04
- U2: footprint Package_DIP:DIP-16_W7.62mm_Socket -> Package_DIP:DIP-16_W7.62mm
- renumbered C2 to C3
Connections:
- net AB11: now also JP7.1 (Pin_1), U3.13; no longer U1.23 (A11)
- net AB12: now also JP6.1 (Pin_1), U3.3; no longer U1.2 (A12)
- net AB13: now also JP5.1 (Pin_1), U3.1; no longer JP2.4 (Pin_4)
- net GND: now also C2.2, U3.11, U3.5, U3.7 (GND), U3.9
- net VCC: now also C2.1, R1.1, U3.14 (VCC)
- net ~{CS}: now also JP1.1 (Pin_1), JP1.3 (Pin_3), JP1.5 (Pin_5), JP4.1 (Pin_1), R1.2; no longer JP4.2 (Pin_2)
- net ~{OE}: now also JP4.2 (Pin_2); no longer JP1.1 (Pin_1), JP1.3 (Pin_3), JP1.5 (Pin_5), JP4.1 (Pin_1)
- new net: JP6.3 (Pin_3), U3.4
- new net: JP2.4 (Pin_4), JP5.2 (Pin_2)
- new net: JP5.3 (Pin_3), U3.2
- new net: JP7.3 (Pin_3), U3.12
- new net A11: JP7.2 (Pin_2), U1.23 (A11)
- new net A12: JP6.2 (Pin_2), U1.2 (A12)
- no-connect marks 40 -> 43
Other:
- company: (none) -> Plastic Objects Limited
- title: (none) -> PAL-2 ROM Board
- moved on the sheet: C1, C3, J1, J4, JP1, JP2, JP3, JP4, U1, U2
